File: ROMSIMM.sch (KiCad schematic (older format))
At the start: 9 parts, among them J1 Conn_01x30

Commit message: asdsda
Parts:
- removed J1: Conn_01x30, stdpads:Memory_SIMM_30, symbol Connector_Generic:Conn_01x30
- removed U? (x4): 39F040, stdpads:PLCC-32_SMDSocket, symbol stdparts:39F040
- added C5, C6: 2u2, stdpads:C_0603, symbol Device:C_Small
- added J1: ROM, stdpads:MacIIROMSIMM_Edge, symbol Connector_Generic:Conn_02x32_Counter_Clockwise
- added U1: D31-24, stdpads:PLCC-32_SMDSocket, symbol GW_RAM:Flash-512Kx8-PLCC-32
- added U2: D23-16, stdpads:PLCC-32_SMDSocket, symbol GW_RAM:Flash-512Kx8-PLCC-32
- added U3: D15-8, stdpads:PLCC-32_SMDSocket, symbol GW_RAM:Flash-512Kx8-PLCC-32
- added U4: D7-0, stdpads:PLCC-32_SMDSocket, symbol GW_RAM:Flash-512Kx8-PLCC-32
- C1, C2, C3, C4: value 100n -> 10u; footprint stdpads:C_1206 -> stdpads:C_0805
Connections:
- net labels added: A21, A22, ~CS~, ~OE~
- net labels removed: DP, QP, ~CASP~, ~CAS~, ~RAS~
- wire segments 6 -> 14
- no-connect marks 0 -> 1
