File: ROMSIMM.sch (KiCad schematic (older format))
At the start: 40 parts, among them J1 ROM, SW1 ROM Sel., U1 MX29LV640, U10 74AHC245, U11 XC6206P332MR, U12 74LVC1G02GW, U2 MX29LV640, U3 74AHC245, U4 74AHC245, U5 74AHC245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

Commit message: Eliminated one 74AHC245PW
Parts:
- removed U8: 74AHC245, stdpads:TSSOP-20_4.4x6.5mm_P0.65mm, symbol GW_Logic:74245
Connections:
- net RA0 is gone; now on net RA2: U7.9 (A7)
- net RA1 is gone; now on net RA3: U7.8 (A6)
- net A0: no longer U7.11 (B7)
- net A1: no longer U7.12 (B6)
- net A2: now also U7.11 (B7); no longer U7.13 (B5)
- net A3: now also U7.12 (B6); no longer U7.14 (B4)
- net A4: now also U7.13 (B5); no longer U7.15 (B3)
- net A5: now also U7.14 (B4); no longer U7.16 (B2)
- net A6: now also U7.15 (B3); no longer U7.17 (B1)
- net A7: now also U7.16 (B2); no longer U7.18 (B0)
- net A8: now also U9.12 (B6); no longer U9.11 (B7)
- net A9: now also U9.13 (B5); no longer U9.12 (B6)
- net GND: no longer U9.13 (B5)
- net RA2: no longer U7.7 (A5)
- net RA3: no longer U7.6 (A4)
- net RA4: now also U7.7 (A5); no longer U7.5 (A3)
- net RA5: now also U7.6 (A4); no longer U7.4 (A2)
- net RA6: now also U7.5 (A3); no longer U7.3 (A1)
- net RA7: now also U7.4 (A2); no longer U7.2 (A0)
- net RA8: now also U9.8 (A6); no longer U9.9 (A7)
- net RA9: now also U9.7 (A5); no longer U9.8 (A6)
- net R~CS~: now also U7.3 (A1)
- net R~OE~: now also U7.2 (A0)
- net R~WE~: now also U9.9 (A7)
- net ~CS~: now also U7.17 (B1)
- net ~OE~: now also U7.18 (B0)
- net ~WE~: now also U9.11 (B7)
- no-connect marks 9 -> 3
Changed lines of the file:
@@
-$EndComp
-$Comp
-L GW_Logic:74245 U8
-U 1 1 5EC89362
-P 4400 3200
-F 0 "U8" H 4400 3800 50  0000 C CNN
-F 1 "74AHC245" H 4400 2600 50  0000 C CNN
-F 2 "stdpads:TSSOP-20_4.4x6.5mm_P0.65mm" H 4400 2550 50  0001 C TNN
-F 3 "" H 4400 3300 60  0001 C CNN
-F 4 "C132987" H 4400 3200 50  0001 C CNN "LCSC Part"
-	1    4400 3200
-	-1   0    0    -1
-$EndComp
-$Comp
-L power:+3V3 #PWR0128
-U 1 1 5EC8936E
-P 4000 2750
-F 0 "#PWR0128" H 4000 2600 50  0001 C CNN
-F 1 "+3V3" H 4000 2900 50  0000 C CNN
-F 2 "" H 4000 2750 50  0001 C CNN
-F 3 "" H 4000 2750 50  0001 C CNN
-	1    4000 2750
-	-1   0    0    -1
 $EndComp
 $Comp
@@
 	4900 1250 4800 1250
 Text Label 4000 2350 2    50   ~ 0
-A0
+A2
 Text Label 4000 2250 2    50   ~ 0
-A1
+A3
 Text Label 4000 2150 2    50   ~ 0
-A2
+A4
 Text Label 4000 2050 2    50   ~ 0
-A3
+A5
 Text Label 4000 1950 2    50   ~ 0
-A4
+A6
 Text Label 4000 1850 2    50   ~ 0
-A5
-Text Label 4000 1750 2    50   ~ 0
-A6
-Text Label 4000 1650 2    50   ~ 0
 A7
 Text Label 4000 4650 2    50   ~ 0
@@
 Text Label 4000 5550 2    50   ~ 0
 A22
-Text Label 4000 4950 2    50   ~ 0
+Text Label 4000 4850 2    50   ~ 0
 A8
-Text Label 4000 4850 2    50   ~ 0
+Text Label 4000 4750 2    50   ~ 0
 A9
 Text Label 4800 2250 0    50   ~ 0
-RA0
+RA2
 Text Label 4800 2150 0    50   ~ 0
-RA1
+RA3
 Text Label 4800 2050 0    50   ~ 0
-RA2
+RA4
 Text Label 4800 1950 0    50   ~ 0
-RA3
+RA5
 Text Label 4800 1850 0    50   ~ 0
-RA4
+RA6
 Text Label 4800 1750 0    50   ~ 0
-RA5
-Text Label 4800 1650 0    50   ~ 0
-RA6
-Text Label 4800 1550 0    50   ~ 0
 RA7
 $Comp
@@
 $EndComp
 $Comp
-L power:GND #PWR0136
-U 1 1 5EC98E92
-P 4800 3650
-F 0 "#PWR0136" H 4800 3400 50  0001 C CNN
-F 1 "GND" H 4800 3500 50  0000 C CNN
-F 2 "" H 4800 3650 50  0001 C CNN
-F 3 "" H 4800 3650 50  0001 C CNN
-	1    4800 3650
-	-1   0    0    -1
-$EndComp
-$Comp
 L power:GND #PWR0137
 U 1 1 5EC99C6D
@@
 	-1   0    0    -1
 $EndComp
-Text Label 4800 3250 0    50   ~ 0
+Text Label 4800 1650 0    50   ~ 0
 R~CS~
-Text Label 4800 3050 0    50   ~ 0
+Text Label 4800 1550 0    50   ~ 0
 R~OE~
-Text Label 4800 2850 0    50   ~ 0
+Text Label 4800 4850 0    50   ~ 0
 R~WE~
-Text Label 4800 4850 0    50   ~ 0
+Text Label 4800 4750 0    50   ~ 0
 RA8
-Text Label 4800 4750 0    50   ~ 0
-RA9
 Wire Wire Line
 	4800 1450 4800 1250
-$Comp
-L power:GND #PWR0138
-U 1 1 5EC9E4BB
-P 4900 2550
-F 0 "#PWR0138" H 4900 2300 50  0001 C CNN
-F 1 "GND" H 4900 2400 50  0000 C CNN
-F 2 "" H 4900 2550 50  0001 C CNN
-F 3 "" H 4900 2550 50  0001 C CNN
-	1    4900 2550
-	-1   0    0    -1
-$EndComp
-Wire Wire Line
-	4900 2550 4800 2550
-Wire Wire Line
-	4800 2750 4800 2550
 $Comp
 L power:GND #PWR0139
@@
 Text Label 4800 5850 0    50   ~ 0
 RA18
-Text Label 4000 2950 2    50   ~ 0
+Text Label 4000 4950 2    50   ~ 0
 ~WE~
-Text Label 4000 3150 2    50   ~ 0
+Text Label 4000 1650 2    50   ~ 0
 ~OE~
-Text Label 4000 3350 2    50   ~ 0
+Text Label 4000 1750 2    50   ~ 0
 ~CS~
 $Comp
@@
 	8350 1600 8650 1600
 Connection ~ 8650 1600
-$Comp
-L power:GND #PWR0149
-U 1 1 5EC0D3D0
-P 3800 4750
-F 0 "#PWR0149" H 3800 4500 50  0001 C CNN
-F 1 "GND" H 3800 4600 50  0000 C CNN
-F 2 "" H 3800 4750 50  0001 C CNN
-F 3 "" H 3800 4750 50  0001 C CNN
-	1    3800 4750
-	-1   0    0    -1
-$EndComp
-Wire Wire Line
-	3800 4750 4000 4750
-$Comp
-L power:GND #PWR0150
-U 1 1 5EC0F52D
-P 3800 3650
-F 0 "#PWR0150" H 3800 3400 50  0001 C CNN
-F 1 "GND" H 3800 3500 50  0000 C CNN
-F 2 "" H 3800 3650 50  0001 C CNN
-F 3 "" H 3800 3650 50  0001 C CNN
-	1    3800 3650
-	-1   0    0    -1
-$EndComp
-Wire Wire Line
-	4000 3650 3800 3650
-Wire Wire Line
-	3800 3650 3800 3550
-Wire Wire Line
-	3800 3050 4000 3050
-Connection ~ 3800 3650
-Wire Wire Line
-	4000 3250 3800 3250
-Connection ~ 3800 3250
-Wire Wire Line
-	3800 3250 3800 3050
-Wire Wire Line
-	4000 3450 3800 3450
-Connection ~ 3800 3450
-Wire Wire Line
-	3800 3450 3800 3250
-Wire Wire Line
-	3800 3550 4000 3550
-Connection ~ 3800 3550
-Wire Wire Line
-	3800 3550 3800 3450
-NoConn ~ 4800 2950
-NoConn ~ 4800 3150
-NoConn ~ 4800 3350
-NoConn ~ 4800 3450
-NoConn ~ 4800 3550
-NoConn ~ 4800 4650
 Wire Wire Line
 	2500 2850 2600 2850
@@
 	-1   0    0    -1
 $EndComp
-$Comp
-L GW_Logic:74245 U9
-U 1 1 5EC8934F
-P 4400 4500
-F 0 "U9" H 4400 5100 50  0000 C CNN
-F 1 "74AHC245" H 4400 3900 50  0000 C CNN
-F 2 "stdpads:TSSOP-20_4.4x6.5mm_P0.65mm" H 4400 3850 50  0001 C TNN
-F 3 "" H 4400 4600 60  0001 C CNN
-F 4 "C132987" H 4400 4500 50  0001 C CNN "LCSC Part"
-	1    4400 4500
-	-1   0    0    -1
-$EndComp
-Wire Wire Line
-	3900 2650 3900 2850
-Wire Wire Line
-	3800 2650 3900 2650
-$Comp
-L power:GND #PWR0131
-U 1 1 5EC5BB53
-P 3800 2650
-F 0 "#PWR0131" H 3800 2400 50  0001 C CNN
-F 1 "GND" H 3800 2500 50  0000 C CNN
-F 2 "" H 3800 2650 50  0001 C CNN
-F 3 "" H 3800 2650 50  0001 C CNN
-	1    3800 2650
-	1    0    0    -1
-$EndComp
-Wire Wire Line
-	3900 2850 4000 2850
 $Comp
 L power:GND #PWR0153
@@
 	1    0    0    -1
 $EndComp
+$Comp
+L GW_Logic:74245 U9
+U 1 1 5EC8934F
+P 4400 4500
+F 0 "U9" H 4400 5100 50  0000 C CNN
+F 1 "74AHC245" H 4400 3900 50  0000 C CNN
+F 2 "stdpads:TSSOP-20_4.4x6.5mm_P0.65mm" H 4400 3850 50  0001 C TNN
+F 3 "" H 4400 4600 60  0001 C CNN
+F 4 "C132987" H 4400 4500 50  0001 C CNN "LCSC Part"
+	1    4400 4500
+	-1   0    0    -1
+$EndComp
+Text Label 4800 4650 0    50   ~ 0
+RA9
 $EndSCHEMATC

Commit message: Migrate to KiCAD 6
Parts:
- added R4: 3k3, stdpads:R_0603, symbol Device:R_Small
- SW1: footprint stdpads:SW_DIP_SPSTx02_Slide_DSHP02TS_P1.27mm -> stdpads:SW_DIP_SPSTx03_Slide_DSHP03TS_P1.27mm; symbol Switch:SW_DIP_x02 -> Switch:SW_DIP_x03
Connections:
- net +3V3: now also R4.2
- net GND: now also SW1.3; no longer SW1.2
- net RA21: now also SW1.1; no longer U1.9 (A19), U2.9 (A19)
- net RA22: now also SW1.2; no longer SW1.1
- net RA22sw: now also R1.1, SW1.5; no longer R2.1, SW1.4
- net RA23: now also R2.1, SW1.4; no longer R1.1, SW1.3
- new net RA21sw: R4.1, SW1.6, U1.9 (A19), U2.9 (A19)
Other:
- moved on the sheet: R1, R2, R3, U12
Changed lines of the file:
@@
 RA22sw
 Text Label 8600 4700 2    50   ~ 0
-RA21
+RA21sw
 Text Label 8600 4600 2    50   ~ 0
 RA20
@@
 RA22sw
 Text Label 7050 4700 2    50   ~ 0
-RA21
+RA21sw
 Text Label 7050 4600 2    50   ~ 0
 RA20
@@
 L GW_Logic:741G02GW U12
 U 1 1 5EF4BDF5
-P 5700 3250
-F 0 "U12" H 5700 3500 50  0000 C CNN
-F 1 "74LVC1G02GW" H 5700 3000 50  0000 C CNN
-F 2 "stdpads:SOT-353" H 5700 2950 50  0001 C TNN
-F 3 "" H 5700 3050 60  0001 C CNN
-F 4 "C353856" H 5700 3250 50  0001 C CNN "LCSC Part"
-	1    5700 3250
-	1    0    0    -1
-$EndComp
-Text Label 5300 3150 2    50   ~ 0
+P 5700 3350
+F 0 "U12" H 5700 3600 50  0000 C CNN
+F 1 "74LVC1G02GW" H 5700 3100 50  0000 C CNN
+F 2 "stdpads:SOT-353" H 5700 3050 50  0001 C TNN
+F 3 "" H 5700 3150 60  0001 C CNN
+F 4 "C353856" H 5700 3350 50  0001 C CNN "LCSC Part"
+	1    5700 3350
+	1    0    0    -1
+$EndComp
+Text Label 5300 3250 2    50   ~ 0
 ~CS~
 $Comp
 L power:+3V3 #PWR0154
 U 1 1 5EF4CD76
-P 6100 3150
-F 0 "#PWR0154" H 6100 3000 50  0001 C CNN
-F 1 "+3V3" H 6100 3300 50  0000 C CNN
-F 2 "" H 6100 3150 50  0001 C CNN
-F 3 "" H 6100 3150 50  0001 C CNN
-	1    6100 3150
+P 6100 3250
+F 0 "#PWR0154" H 6100 3100 50  0001 C CNN
+F 1 "+3V3" H 6100 3400 50  0000 C CNN
+F 2 "" H 6100 3250 50  0001 C CNN
+F 3 "" H 6100 3250 50  0001 C CNN
+	1    6100 3250
 	-1   0    0    -1
 $EndComp
@@
 L power:GND #PWR0155
 U 1 1 5EF4D490
-P 5300 3350
-F 0 "#PWR0155" H 5300 3100 50  0001 C CNN
-F 1 "GND" H 5300 3200 50  0000 C CNN
-F 2 "" H 5300 3350 50  0001 C CNN
-F 3 "" H 5300 3350 50  0001 C CNN
-	1    5300 3350
-	-1   0    0    -1
-$EndComp
-Text Label 6500 3350 0    50   ~ 0
+P 5300 3450
+F 0 "#PWR0155" H 5300 3200 50  0001 C CNN
+F 1 "GND" H 5300 3300 50  0000 C CNN
+F 2 "" H 5300 3450 50  0001 C CNN
+F 3 "" H 5300 3450 50  0001 C CNN
+	1    5300 3450
+	-1   0    0    -1
+$EndComp
+Text Label 6500 3450 0    50   ~ 0
 DdirR
-Text Label 5300 3250 2    50   ~ 0
+Text Label 5300 3350 2    50   ~ 0
 ~OE~
 $Comp
 L Device:R_Small R3
 U 1 1 5EFDEB5D
-P 6400 3350
-F 0 "R3" V 6350 3350 50  0000 C BNN
-F 1 "100" V 6450 3350 50  0000 C TNN
-F 2 "stdpads:R_0603" H 6400 3350 50  0001 C CNN
-F 3 "~" H 6400 3350 50  0001 C CNN
-F 4 "C22775" V 6400 3350 50  0001 C CNN "LCSC Part"
-	1    6400 3350
+P 6400 3450
+F 0 "R3" V 6350 3450 50  0000 C BNN
+F 1 "100" V 6450 3450 50  0000 C TNN
+F 2 "stdpads:R_0603" H 6400 3450 50  0001 C CNN
+F 3 "~" H 6400 3450 50  0001 C CNN
+F 4 "C22775" V 6400 3450 50  0001 C CNN "LCSC Part"
+	1    6400 3450
 	0    1    1    0
 $EndComp
-Text Label 6100 3350 0    50   ~ 0
+Text Label 6100 3450 0    50   ~ 0
 Ddir
 Wire Wire Line
-	6100 3350 6300 3350
-Text Label 6500 2550 0    50   ~ 0
+	6100 3450 6300 3450
+Text Label 6650 2550 0    50   ~ 0
 RA23
 $Comp
 L Device:R_Small R1
 U 1 1 CB6D6B90
-P 6100 2300
-F 0 "R1" H 6159 2346 50  0000 L CNN
-F 1 "3k3" H 6159 2255 50  0000 L CNN
-F 2 "stdpads:R_0603" H 6100 2300 50  0001 C CNN
-F 3 "~" H 6100 2300 50  0001 C CNN
-F 4 "C22978" H 6100 2300 50  0001 C CNN "LCSC Part"
-	1    6100 2300
+P 6150 2200
+F 0 "R1" H 6209 2246 50  0000 L CNN
+F 1 "3k3" H 6209 2155 50  0000 L CNN
+F 2 "stdpads:R_0603" H 6150 2200 50  0001 C CNN
+F 3 "~" H 6150 2200 50  0001 C CNN
+F 4 "C22978" H 6150 2200 50  0001 C CNN "LCSC Part"
+	1    6150 2200
 	1    0    0    1
 $EndComp
@@
 L power:+3V3 #PWR0151
 U 1 1 CB6D6B97
-P 6400 2200
-F 0 "#PWR0151" H 6400 2050 50  0001 C CNN
-F 1 "+3V3" H 6400 2350 50  0000 C CNN
-F 2 "" H 6400 2200 50  0001 C CNN
-F 3 "" H 6400 2200 50  0001 C CNN
-	1    6400 2200
-	-1   0    0    -1
-$EndComp
-Text Label 6500 2450 0    50   ~ 0
+P 6450 2100
+F 0 "#PWR0151" H 6450 1950 50  0001 C CNN
+F 1 "+3V3" H 6450 2250 50  0000 C CNN
+F 2 "" H 6450 2100 50  0001 C CNN
+F 3 "" H 6450 2100 50  0001 C CNN
+	1    6450 2100
+	-1   0    0    -1
+$EndComp
+Text Label 6650 2450 0    50   ~ 0
 RA22sw
-Wire Wire Line
-	6500 2450 6400 2450
 $Comp
 L Device:R_Small R2
 U 1 1 CB6E14B2
-P 6400 2300
-F 0 "R2" H 6459 2346 50  0000 L CNN
-F 1 "3k3" H 6459 2255 50  0000 L CNN
-F 2 "stdpads:R_0603" H 6400 2300 50  0001 C CNN
-F 3 "~" H 6400 2300 50  0001 C CNN
-F 4 "C22978" H 6400 2300 50  0001 C CNN "LCSC Part"
-	1    6400 2300
+P 6450 2200
+F 0 "R2" H 6509 2246 50  0000 L CNN
+F 1 "3k3" H 6509 2155 50  0000 L CNN
+F 2 "stdpads:R_0603" H 6450 2200 50  0001 C CNN
+F 3 "~" H 6450 2200 50  0001 C CNN
+F 4 "C22978" H 6450 2200 50  0001 C CNN "LCSC Part"
+	1    6450 2200
 	1    0    0    1
 $EndComp
 Wire Wire Line
-	6000 2550 6100 2550
-Wire Wire Line
-	6400 2450 6400 2400
-Wire Wire Line
-	6100 2550 6500 2550
-Connection ~ 6100 2550
-Wire Wire Line
-	6100 2550 6100 2400
-Connection ~ 6400 2450
-Wire Wire Line
-	6400 2450 6000 2450
-Wire Wire Line
-	6400 2200 6100 2200
+	6450 2100 6150 2100
 $Comp
 L power:GND #PWR0152
 U 1 1 CB700278
-P 5400 2550
-F 0 "#PWR0152" H 5400 2300 50  0001 C CNN
-F 1 "GND" H 5400 2400 50  0000 C CNN
-F 2 "" H 5400 2550 50  0001 C CNN
-F 3 "" H 5400 2550 50  0001 C CNN
-	1    5400 2550
-	-1   0    0    -1
-$EndComp
-Text Label 5400 2450 2    50   ~ 0
+P 5150 2550
+F 0 "#PWR0152" H 5150 2300 50  0001 C CNN
+F 1 "GND" H 5150 2400 50  0000 C CNN
+F 2 "" H 5150 2550 50  0001 C CNN
+F 3 "" H 5150 2550 50  0001 C CNN
+	1    5150 2550
+	-1   0    0    -1
+$EndComp
+Text Label 5150 2450 2    50   ~ 0
 RA22
 $Comp
@@
 	-1   0    0    -1
 $EndComp
-Connection ~ 6400 2200
-$Comp
-L Switch:SW_DIP_x02 SW1
-U 1 1 CB6D2346
-P 5700 2550
-F 0 "SW1" H 5700 2800 50  0000 C CNN
-F 1 "ROM Sel." H 5700 2400 50  0000 C CNN
-F 2 "stdpads:SW_DIP_SPSTx02_Slide_DSHP02TS_P1.27mm" H 5700 2550 50  0001 C CNN
-F 3 "~" H 5700 2550 50  0001 C CNN
-F 4 "C319052" H 5700 2550 50  0001 C CNN "LCSC Part"
-	1    5700 2550
-	1    0    0    -1
-$EndComp
+Connection ~ 6450 2100
 $Comp
 L GW_Logic:74245 U9
@@
 Text Label 4800 4650 0    50   ~ 0
 RA9
+$Comp
+L Switch:SW_DIP_x03 SW1
+U 1 1 CB6D2346
+P 5450 2550
+F 0 "SW1" H 5450 2800 50  0000 C CNN
+F 1 "ROM Sel." H 5450 2400 50  0000 C CNN
+F 2 "stdpads:SW_DIP_SPSTx03_Slide_DSHP03TS_P1.27mm" H 5450 2550 50  0001 C CNN
+F 3 "~" H 5450 2550 50  0001 C CNN
+F 4 "C319052" H 5450 2550 50  0001 C CNN "LCSC Part"
+	1    5450 2550
+	1    0    0    -1
+$EndComp
+Text Label 5150 2350 2    50   ~ 0
+RA21
+$Comp
+L Device:R_Small R4
+U 1 1 6229CD7C
+P 5850 2200
+F 0 "R4" H 5909 2246 50  0000 L CNN
+F 1 "3k3" H 5909 2155 50  0000 L CNN
+F 2 "stdpads:R_0603" H 5850 2200 50  0001 C CNN
+F 3 "~" H 5850 2200 50  0001 C CNN
+F 4 "C22978" H 5850 2200 50  0001 C CNN "LCSC Part"
+	1    5850 2200
+	1    0    0    1
+$EndComp
+Wire Wire Line
+	6150 2100 5850 2100
+Wire Wire Line
+	5850 2350 5850 2300
+Connection ~ 6150 2100
+Wire Wire Line
+	5750 2550 6450 2550
+Wire Wire Line
+	5750 2450 6150 2450
+Wire Wire Line
+	5750 2350 5850 2350
+Wire Wire Line
+	6150 2300 6150 2450
+Connection ~ 6150 2450
+Wire Wire Line
+	6150 2450 6650 2450
+Wire Wire Line
+	6450 2300 6450 2550
+Connection ~ 6450 2550
+Wire Wire Line
+	6450 2550 6650 2550
+Text Label 6650 2350 0    50   ~ 0
+RA21sw
+Wire Wire Line
+	6650 2350 5850 2350
+Connection ~ 5850 2350
 $EndSCHEMATC
