File: ROMSIMM.kicad_pcb (KiCad board)
At the start: 4 copper layers, 97.8 x 25 mm, 40 parts, among them J1 ROM, SW1 ROM Sel., U1 MX29LV640, U10 74AHC245, U11 XC6206P332MR, U12 74LVC1G02GW, U2 MX29LV640, U3 74AHC245, U4 74AHC245, U5 74AHC245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

Commit message: Eliminated one 74AHC245PW
Parts:
- removed U8: 74AHC245, stdpads:TSSOP-20_4.4x6.5mm_P0.65mm
Connections:
- U7 pad 11: /A0 -> /A2
- U7 pad 12: /A1 -> /A3
- U7 pad 13: /A2 -> /A4
- U7 pad 14: /A3 -> /A5
- U7 pad 15: /A4 -> /A6
- U7 pad 16: /A5 -> /A7
- U7 pad 17: /A6 -> /~CS~
- U7 pad 18: /A7 -> /~OE~
- U7 pad 2: /RA7 -> /R~OE~
- U7 pad 3: /RA6 -> /R~CS~
- U7 pad 4: /RA5 -> /RA7
- U7 pad 5: /RA4 -> /RA6
- U7 pad 6: /RA3 -> /RA5
- U7 pad 7: /RA2 -> /RA4
- U7 pad 8: /RA1 -> /RA3
- U7 pad 9: /RA0 -> /RA2
- U9 pad 11: /A8 -> /~WE~
- U9 pad 12: /A9 -> /A8
- U9 pad 13: GND -> /A9
- U9 pad 7: Net-(U9-Pad7) -> /RA9
- U9 pad 8: /RA9 -> /RA8
- U9 pad 9: /RA8 -> /R~WE~
Routing:
- net /~WE~: track 2.12 -> 35.4 mm, vias 0 -> 1
- net GND: track 97.6 -> 84.9 mm, vias 159 -> 153
- net /~OE~: track 12.4 -> 24.6 mm
- net /R~OE~: track 69.7 -> 80.1 mm
- net /~CS~: track 10.2 -> 19.6 mm, vias 0 -> 1
- net /R~CS~: track 71.6 -> 80.2 mm
- net /A1: track 6.38 -> 0.00 mm, vias 1 -> 0
- net /A0: track 4.47 -> 0.00 mm, vias 1 -> 0
- net /R~WE~: track 56.0 -> 53.3 mm, vias 2 -> 3
- net /A7: track 9.37 -> 12.0 mm
- net /A8: track 9.16 -> 11.5 mm
- net +5V: track 164.2 -> 166.3 mm
- net /A6: track 7.30 -> 9.20 mm
- net /RA2: track 83.5 -> 85.2 mm
- net /RA6: track 54.2 -> 55.5 mm
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Other:
- board text added: "ZK, GF"
