File: SIMM8MB.4402A/ROMSIMM.kicad_pcb (KiCad board)
At the start: 4 copper layers, 97.8 x 25 mm, 34 parts, among them J1 ROM, U1 MX29LV320, U10 74AHC245, U11 LD1117S33, U2 MX29LV320, U3 74AHC245, U4 74AHC245, U5 74AHC245, U6 74AHC245, U7 74AHC245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

Commit message: 8MB stitching fix
Routing:
- net GND: track 76.4 -> 75.4 mm, vias 167 -> 166
Changed lines of the file:
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@@
     (thickness 1.6)
     (drawings 23)
-    (tracks 1262)
+    (tracks 1259)
     (zones 0)
     (modules 34)
@@
   (via (at 79.1 112.85) (size 0.5) (drill 0.2) (layers F.Cu B.Cu) (net 7))
   (segment (start 79.1 113.75) (end 79.1 112.85) (width 0.5) (layer F.Cu) (net 7))
-  (via (at 108.25 114.45) (size 0.5) (drill 0.2) (layers F.Cu B.Cu) (net 7))
-  (segment (start 109.2 114.45) (end 108.25 114.45) (width 0.25) (layer F.Cu) (net 7))
   (via (at 110.15 114.45) (size 0.5) (drill 0.2) (layers F.Cu B.Cu) (net 7))
   (segment (start 109.2 114.45) (end 110.15 114.45) (width 0.25) (layer F.Cu) (net 7))
@@
   (segment (start 89.69 113.95) (end 88.75 113.95) (width 0.15) (layer F.Cu) (net 95))
   (via (at 88.75 113.95) (size 0.5) (drill 0.2) (layers F.Cu B.Cu) (net 95))
-  (segment (start 110.5 113.65) (end 107.9 113.65) (width 0.15) (layer In2.Cu) (net 95))
-  (segment (start 107.2 113.95) (end 88.75 113.95) (width 0.15) (layer In2.Cu) (net 95))
-  (segment (start 110.8 113.95) (end 110.5 113.65) (width 0.15) (layer In2.Cu) (net 95))
-  (segment (start 107.4 114.15) (end 107.2 113.95) (width 0.15) (layer In2.Cu) (net 95))
-  (segment (start 107.9 113.65) (end 107.4 114.15) (width 0.15) (layer In2.Cu) (net 95))
-  (segment (start 131.55 113.95) (end 110.8 113.95) (width 0.15) (layer In2.Cu) (net 95))
   (segment (start 84.25 118.85) (end 85 118.85) (width 0.15) (layer F.Cu) (net 95))
   (segment (start 85 118.85) (end 85.95 117.9) (width 0.15) (layer F.Cu) (net 95))
@@
   (segment (start 83.5 117.2) (end 83.5 118.1) (width 0.15) (layer F.Cu) (net 95))
   (segment (start 85.95 116.5) (end 88.5 113.95) (width 0.15) (layer F.Cu) (net 95))
+  (segment (start 107.6 113.95) (end 88.75 113.95) (width 0.15) (layer In2.Cu) (net 95))
+  (segment (start 107.9 113.65) (end 107.6 113.95) (width 0.15) (layer In2.Cu) (net 95))
+  (segment (start 110.5 113.65) (end 107.9 113.65) (width 0.15) (layer In2.Cu) (net 95))
+  (segment (start 110.8 113.95) (end 110.5 113.65) (width 0.15) (layer In2.Cu) (net 95))
+  (segment (start 131.55 113.95) (end 110.8 113.95) (width 0.15) (layer In2.Cu) (net 95))
   (via (at 133.45 114.45) (size 0.5) (drill 0.2) (layers F.Cu B.Cu) (net 96))
   (segment (start 132.49 114.45) (end 133.45 114.45) (width 0.15) (layer F.Cu) (net 96))
