File: SIMMuSD.4403A/ROMSIMM.kicad_pcb (KiCad board)
At the start: 4 copper layers, 97.8 x 26.9 mm, 31 parts, among them J1 ROM, U1 MX29LV640, U11 LD1117S33, U5 M5LV-TQFP-144

Commit message: Update ROMSIMM.kicad_pcb
Parts:
- removed C10, C4, C5, C6, C7, C8: 2u2, stdpads:C_0603
- removed the REF** at (131.5, 85.4)
- removed the REF** at (116.3, 113.0)
- removed U1: MX29LV640, stdpads:TSOP-I-48_18.4x12mm_P0.5mm
- removed U5: M5LV-TQFP-144, stdpads:TQFP-144_20x20mm_P0.5mm
- added REF**: LQFP-64-1EP_10x10mm_P0.5mm_EP5x5mm, Package_QFP:LQFP-64-1EP_10x10mm_P0.5mm_EP5x5mm, F.Cu at (158.4, 110.5)
- added REF**: NXP_DHVFQFN-20_SOT764-1, stdpads:NXP_DHVFQFN-20_SOT764-1, F.Cu at (88.5, 121.2)
- added REF**: NXP_DHVFQFN-20_SOT764-1, stdpads:NXP_DHVFQFN-20_SOT764-1, F.Cu at (82.2, 121.5)
- added REF**: TSOP-I-48_18.4x12mm_P0.5mm, stdpads:TSOP-I-48_18.4x12mm_P0.5mm, F.Cu at (131.8, 113.2)
- added REF**: TSOP-I-48_18.4x12mm_P0.5mm, stdpads:TSOP-I-48_18.4x12mm_P0.5mm, F.Cu at (144.8, 113.2)
- added REF**: NXP_DHVFQFN-20_SOT764-1, stdpads:NXP_DHVFQFN-20_SOT764-1, F.Cu at (161.6, 121.3)
- added REF**: NXP_DHVFQFN-20_SOT764-1, stdpads:NXP_DHVFQFN-20_SOT764-1, F.Cu at (114.3, 121.3)
- added REF**: NXP_DHVFQFN-20_SOT764-1, stdpads:NXP_DHVFQFN-20_SOT764-1, F.Cu at (107.8, 121.3)
- added REF**: NXP_DHVFQFN-20_SOT764-1, stdpads:NXP_DHVFQFN-20_SOT764-1, F.Cu at (155.0, 121.2)
- added REF**: NXP_DHVFQFN-20_SOT764-1, stdpads:NXP_DHVFQFN-20_SOT764-1, F.Cu at (101.5, 121.3)
- added REF**: NXP_DHVFQFN-20_SOT764-1, stdpads:NXP_DHVFQFN-20_SOT764-1, F.Cu at (94.8, 121.2)
Routing:
- net GND: track 56.0 -> 3.05 mm, vias 67 -> 21
- net +3V3: track 47.0 -> 15.0 mm, vias 35 -> 8
- net /D15: track 13.6 -> 0.00 mm
- net /A8: track 12.1 -> 0.00 mm, vias 1 -> 0
- net /D22: track 9.62 -> 0.00 mm
- net /A9: track 8.41 -> 0.00 mm, vias 1 -> 0
- net /D21: track 8.06 -> 0.00 mm
- net /D20: track 7.07 -> 0.00 mm
- net /D19: track 6.07 -> 0.00 mm
- net /D18: track 5.64 -> 0.00 mm
- net /D17: track 5.39 -> 0.00 mm
- net /A7: track 2.01 -> 0.00 mm, vias 1 -> 0
- net /D31: track 2.01 -> 0.00 mm, vias 1 -> 0
- net /D29: track 2.01 -> 0.00 mm, vias 1 -> 0
- net /A17: track 2.00 -> 0.00 mm
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