File: SIMMuSD.4404A/ROMSIMM.kicad_pcb (KiCad board)
At the start: 4 copper layers, 97.8 x 26.9 mm, 32 parts, among them J1 ROM, U11 LD1117S33

Commit message: More uSD
Parts:
- removed the R1 at (158.5, 133.2)
- removed REF** (x7): NXP_DHVFQFN-20_SOT764-1, stdpads:NXP_DHVFQFN-20_SOT764-1
- removed REF**: Tag-Connect_TC2050-IDC-FP_2x05_P1.27mm_Vertical, Connector:Tag-Connect_TC2050-IDC-FP_2x05_P1.27mm_Vertical
- removed REF**: Molex_473521001_microSD, stdpads:Molex_473521001_microSD
- removed REF** (x2): TSOP-I-48_18.4x12mm_P0.5mm, stdpads:TSOP-I-48_18.4x12mm_P0.5mm
- added C10: 2u2, stdpads:C_0603, F.Cu at (142.0, 122.2)
- added C16: 2u2, stdpads:C_0603, F.Cu at (128.3, 109.1)
- added C17, C19, C20: 2u2, stdpads:C_0603, F.Cu at (120.7, 137.7)
- added C18: 2u2, stdpads:C_0603, F.Cu at (171.5, 128.7)
- added C21: 2u2, stdpads:C_0603, F.Cu at (171.5, 131.1)
- added C4: 10u, stdpads:C_0805, F.Cu at (66.3, 102.8)
- added C5: 2u2, stdpads:C_0603, F.Cu at (82.3, 122.2)
- added C6: 2u2, stdpads:C_0603, F.Cu at (95.0, 122.2)
- added C7: 2u2, stdpads:C_0603, F.Cu at (105.2, 122.2)
- added C8: 2u2, stdpads:C_0603, F.Cu at (122.5, 122.2)
- added C9: 2u2, stdpads:C_0603, F.Cu at (131.8, 122.2)
- added J2: Micro_SD_SingleDet, stdpads:Molex_473521001_microSD, F.Cu at (158.3, 109.8)
- added J3: Tag-Connect_TC2050-IDC-NL_2x05_P1.27mm_Vertical, Connector:Tag-Connect_TC2050-IDC-NL_2x05_P1.27mm_Vertical, F.Cu at (166.1, 110.3)
- added R1: 3k3, stdpads:R_0805, F.Cu at (147.2, 110.6)
- added R1: 3k3, stdpads:R_0805, F.Cu at (160.9, 121.4)
- added U10: 74AHC245BQ, stdpads:NXP_DHVFQFN-20_SOT764-1, F.Cu at (156.2, 121.8)
- added U12: 50M, stdpads:Crystal_SMD_3225-4Pin_3.2x2.5mm, F.Cu at (145.2, 106.8)
- added U2: MX29LV640, stdpads:TSOP-I-48_18.4x12mm_P0.5mm, F.Cu at (90.8, 109.8)
- added U3: MX29LV640, stdpads:TSOP-I-48_18.4x12mm_P0.5mm, F.Cu at (115.0, 109.8)
- added U4: 74AHC245BQ, stdpads:NXP_DHVFQFN-20_SOT764-1, F.Cu at (86.3, 121.8)
- added U5: 74AHC245BQ, stdpads:NXP_DHVFQFN-20_SOT764-1, F.Cu at (99.0, 121.8)
- added U6: 74AHC245BQ, stdpads:NXP_DHVFQFN-20_SOT764-1, F.Cu at (109.2, 121.8)
- added U7: 74AHC245BQ, stdpads:NXP_DHVFQFN-20_SOT764-1, F.Cu at (126.5, 121.8)
- added U9: 74AHC245BQ, stdpads:NXP_DHVFQFN-20_SOT764-1, F.Cu at (146.1, 121.8)
- C1, C2: value 2u2 -> 10u; footprint stdpads:C_0603 -> stdpads:C_0805
- U1: renamed from REF**; value LQFP-64-1EP_10x10mm_P0.5mm_EP5x5mm -> 5M80ZE68
- U8: renamed from REF**; value NXP_DHVFQFN-20_SOT764-1 -> 74AHC245BQ
- moved C2 81.0 mm to (79.0, 117.7)
- moved C1 80.3 mm to (79.0, 122.2)
- moved C12 62.8 mm to (102.5, 104.8), turned to 270 degrees
- moved C15 41.9 mm to (129.5, 103.7), turned to 180 degrees
- moved C14 33.4 mm to (142.8, 103.7)
- moved C13 26.5 mm to (144.6, 110.6), turned to 270 degrees
- moved U1 22.3 mm to (136.2, 109.6), turned to 180 degrees
- moved U8 21.6 mm to (135.9, 121.8)
- moved C3 21.2 mm to (140.3, 122.2), turned to 90 degrees
- moved C11 12.6 mm to (152.2, 122.2), turned to 270 degrees
- moved FID1 0.89 mm to (75.9, 103.3)
- moved FID4 0.89 mm to (165.4, 103.3)
- moved H1 0.89 mm to (73.4, 103.3)
- moved H4 0.89 mm to (167.9, 103.3)
- moved U11 0.21 mm to (76.5, 110.2)
- renumbered C9 to C15
Connections:
- U1 pad 1: (no net) -> Net-(U1-Pad1)
- U1 pad 10: (no net) -> Net-(U1-Pad10)
- U1 pad 11: (no net) -> Net-(U1-Pad11)
- U1 pad 12: (no net) -> Net-(U1-Pad12)
- U1 pad 13: (no net) -> Net-(U1-Pad13)
- U1 pad 14: (no net) -> /TMS
- U1 pad 15: (no net) -> /TDI
- U1 pad 16: (no net) -> /TCK
- U1 pad 17: (no net) -> /TDO
- U1 pad 18: (no net) -> Net-(U1-Pad18)
- U1 pad 19: (no net) -> Net-(U1-Pad19)
- U1 pad 2: (no net) -> Net-(U1-Pad2)
- U1 pad 20: (no net) -> Net-(U1-Pad20)
- U1 pad 21: (no net) -> Net-(U1-Pad21)
- U1 pad 22: (no net) -> Net-(U1-Pad22)
- U1 pad 23: (no net) -> +3V3
- U1 pad 24: (no net) -> Net-(U1-Pad24)
- U1 pad 25: (no net) -> Net-(U1-Pad25)
- U1 pad 26: (no net) -> Net-(U1-Pad26)
- U1 pad 27: (no net) -> Net-(U1-Pad27)
- U1 pad 28: (no net) -> Net-(U1-Pad28)
- U1 pad 29: (no net) -> Net-(U1-Pad29)
- U1 pad 3: (no net) -> Net-(U1-Pad3)
- U1 pad 30: (no net) -> Net-(U1-Pad30)
- U1 pad 31: (no net) -> Net-(U1-Pad31)
- U1 pad 32: (no net) -> /RD31
- U1 pad 33: (no net) -> /RD30
- U1 pad 34: (no net) -> /RD23
- U1 pad 35: (no net) -> /RD22
- U1 pad 36: (no net) -> /RD21
- U1 pad 37: (no net) -> Net-(U1-Pad37)
- U1 pad 38: (no net) -> Net-(U1-Pad38)
- U1 pad 39: (no net) -> +3V3
- U1 pad 4: (no net) -> Net-(U1-Pad4)
- U1 pad 40: (no net) -> /RD28
- U1 pad 41: (no net) -> +3V3
- U1 pad 42: (no net) -> Net-(U1-Pad42)
- U1 pad 43: (no net) -> Net-(U1-Pad43)
- U1 pad 44: (no net) -> /RD29
- U1 pad 45: (no net) -> /RD20
- U1 pad 46: (no net) -> /RD27
- U1 pad 47: (no net) -> /RD19
- U1 pad 48: (no net) -> /RD26
- U1 pad 49: (no net) -> /RD18
- U1 pad 5: (no net) -> Net-(U1-Pad5)
- U1 pad 50: (no net) -> /RD25
- U1 pad 51: (no net) -> /RD17
- U1 pad 52: (no net) -> /RD24
- U1 pad 53: (no net) -> /RD16
- U1 pad 54: (no net) -> /R~OE~
- U1 pad 55: (no net) -> /R~CS~
- U1 pad 56: (no net) -> /R~CS~g
- U1 pad 57: (no net) -> +3V3
- U1 pad 58: (no net) -> /RA2
- U1 pad 59: (no net) -> /RA18
- U1 pad 6: (no net) -> +3V3
- U1 pad 60: (no net) -> /RA19
- U1 pad 61: (no net) -> /RA20
- U1 pad 62: (no net) -> /RA21
- U1 pad 63: (no net) -> /RA22
- U1 pad 64: (no net) -> /R~WE~
- U1 pad 65: (no net) -> GND
- U1 pad 7: (no net) -> /C50M
- U1 pad 8: (no net) -> +3V3
- U1 pad 9: (no net) -> Net-(U1-Pad9)
- U8 pad 1: (no net) -> +3V3
- U8 pad 10: (no net) -> GND
- U8 pad 11: (no net) -> /R~WE~
- U8 pad 12: (no net) -> /RA22
- U8 pad 13: (no net) -> /RA21
- U8 pad 14: (no net) -> /RA20
- U8 pad 15: (no net) -> /RA19
- U8 pad 16: (no net) -> /RA18
- U8 pad 17: (no net) -> /RA17
- U8 pad 18: (no net) -> /RA16
- U8 pad 19: (no net) -> GND
- U8 pad 2: (no net) -> /A16
- U8 pad 20: (no net) -> +3V3
- U8 pad 21: (no net) -> GND
- U8 pad 3: (no net) -> /A17
- U8 pad 4: (no net) -> /A18
- U8 pad 5: (no net) -> /A19
- U8 pad 6: (no net) -> /A20
- U8 pad 7: (no net) -> /A21
- U8 pad 8: (no net) -> /A22
- U8 pad 9: (no net) -> /~WE~
Routing:
- net +3V3: track 15.0 -> 166.0 mm, vias 8 -> 73
- net +5V: track 0.01 -> 139.4 mm, vias 0 -> 1
- net GND: track 3.05 -> 112.9 mm, vias 21 -> 98
- net /RA16: track 0.00 -> 66.2 mm, vias 0 -> 2
- net /RA21: track 0.00 -> 66.1 mm, vias 0 -> 3
- net /RA17: track 0.00 -> 65.2 mm, vias 0 -> 2
- net /RA18: track 0.00 -> 64.5 mm
- net /RA20: track 0.00 -> 63.8 mm, vias 0 -> 3
- net /R~WE~: track 0.00 -> 63.6 mm, vias 0 -> 3
- net /RA22: track 0.00 -> 62.4 mm, vias 0 -> 3
- net /RA19: track 0.00 -> 61.3 mm, vias 0 -> 3
- net /Ddir: track 0.00 -> 60.7 mm, vias 0 -> 4
- net /RA15: track 0.00 -> 60.1 mm, vias 0 -> 2
- net /RA14: track 0.00 -> 59.0 mm, vias 0 -> 2
- net /RA13: track 0.00 -> 57.3 mm, vias 0 -> 2
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Other:
- board size 97.8 x 26.9 mm -> 97.8 x 26 mm
