File: SIMMuSD.4404A/ROMSIMM.sch (KiCad schematic (older format))
At the start: 28 parts, among them J1 ROM, SW1 ROM Select, U1 MX29LV640, U11 LD1117S33, U5 M5LV-TQFP-144

Commit message: More uSD
Parts:
- removed R1: 3k3, stdpads:R_0805, symbol Device:R_Small
- removed SW1: ROM Select, symbol Switch:SW_DIP_x01
- removed U5: M5LV-TQFP-144, stdpads:TQFP-144_20x20mm_P0.5mm, symbol GW_PLD:M5LV-TQFP-144
- added C15, C16, C17, C18, C19, C20, C21: 2u2, stdpads:C_0603, symbol Device:C_Small
- added J2: Micro_SD_SingleDet, symbol GW_Connector:Micro_SD_SingleDet
- added U1: 5M80ZE68, stdpads:EQFP-64_10x10mm_P0.5mm, symbol GW_PLD:5M80ZE68
- added U10, U4, U5, U6, U7, U8, U9: 74AHC245BQ, stdpads:Nexperia_DHVFQFN-20_SOT764-1, symbol GW_Logic:74245BQ
- added U12: 50M, symbol GW_Logic:Oscillator_4P
- added U3: MX29LV640, stdpads:TSOP-I-48_18.4x12mm_P0.5mm, symbol GW_RAM:Flash-4Mx16-TSOP1-48
- C1, C2, C4: value 2u2 -> 10u; footprint stdpads:C_0603 -> stdpads:C_0805
- renumbered U1 to U2
Connections:
- net labels added: C50M, Ddir, MISO, MOSI, R~CS~g, SCK, SDet, S~CS~, TCK, TDI, TDO, TMS
- net labels removed: Clk, RA0, RA1
- wire segments 70 -> 62
- no-connect marks 2 -> 5
Other:
- moved on the sheet: C1, C10, C11, C12, C13, C14, C2, C3, C4, C5, C6, C7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
