File: ROMSIMM8MB.4402A/ROMSIMM.sch (KiCad schematic (older format))
At the start: 39 parts, among them J1 ROM, SW1 ROM Select, U1 MX29LV320, U10 74AHC245, U11 LD1117S33, U12 74LVC1G02GW, U2 MX29LV320, U3 74AHC245, U4 74AHC245, U5 74AHC245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

Commit message: 8MB SIMM as sent to JLCPCB July 2020
Parts:
- U1, U2: value MX29LV320 -> MX29LV640
Other:
- moved on the sheet: R1, SW1
Changed lines of the file:
@@
 U 1 1 5EBFA0B8
 P 9100 3500
-F 0 "U2" H 9100 4667 50  0000 C CNN
-F 1 "MX29LV320" H 9100 4576 50  0000 C CNN
+F 0 "U2" H 9100 4550 50  0000 C CNN
+F 1 "MX29LV640" H 9100 1750 50  0000 C CNN
 F 2 "stdpads:TSOP-I-48_18.4x12mm_P0.5mm" H 9100 3500 50  0001 C CNN
 F 3 "http://ww1.microchip.com/downloads/en/DeviceDoc/25022B.pdf" H 9100 3500 50  0001 C CNN
@@
 U 1 1 5EBF8A7E
 P 7550 3500
-F 0 "U1" H 7550 4667 50  0000 C CNN
-F 1 "MX29LV320" H 7550 4576 50  0000 C CNN
+F 0 "U1" H 7550 4550 50  0000 C CNN
+F 1 "MX29LV640" H 7550 1750 50  0000 C CNN
 F 2 "stdpads:TSOP-I-48_18.4x12mm_P0.5mm" H 7550 3500 50  0001 C CNN
 F 3 "http://ww1.microchip.com/downloads/en/DeviceDoc/25022B.pdf" H 7550 3500 50  0001 C CNN
@@
 Wire Wire Line
 	3900 2850 4000 2850
-Text Label 5400 950  2    50   ~ 0
+Text Label 5850 1750 2    50   ~ 0
 RA23
 $Comp
 L Device:R_Small R1
 U 1 1 5EC0CD79
-P 5500 850
-F 0 "R1" H 5559 896 50  0000 L CNN
-F 1 "3k3" H 5559 805 50  0000 L CNN
-F 2 "stdpads:R_0805" H 5500 850 50  0001 C CNN
-F 3 "~" H 5500 850 50  0001 C CNN
-	1    5500 850
-	1    0    0    -1
-$EndComp
-Wire Wire Line
-	5400 950  5500 950
+P 5950 1650
+F 0 "R1" H 6009 1696 50  0000 L CNN
+F 1 "3k3" H 6009 1605 50  0000 L CNN
+F 2 "stdpads:R_0805" H 5950 1650 50  0001 C CNN
+F 3 "~" H 5950 1650 50  0001 C CNN
+	1    5950 1650
+	1    0    0    -1
+$EndComp
+Wire Wire Line
+	5850 1750 5950 1750
 $Comp
 L power:+3V3 #PWR0151
 U 1 1 5EC0FA8C
-P 5500 750
-F 0 "#PWR0151" H 5500 600 50  0001 C CNN
-F 1 "+3V3" H 5500 900 50  0000 C CNN
-F 2 "" H 5500 750 50  0001 C CNN
-F 3 "" H 5500 750 50  0001 C CNN
-	1    5500 750
+P 5950 1550
+F 0 "#PWR0151" H 5950 1400 50  0001 C CNN
+F 1 "+3V3" H 5950 1700 50  0000 C CNN
+F 2 "" H 5950 1550 50  0001 C CNN
+F 3 "" H 5950 1550 50  0001 C CNN
+	1    5950 1550
 	-1   0    0    -1
 $EndComp
@@
 L Switch:SW_DIP_x01 SW1
 U 1 1 5EC10C6B
-P 5900 950
-F 0 "SW1" H 5900 1100 50  0000 C CNN
-F 1 "ROM Select" H 5900 800 50  0000 C CNN
-F 2 "Button_Switch_SMD:SW_DIP_SPSTx01_Slide_6.7x4.1mm_W8.61mm_P2.54mm_LowProfile" H 5900 950 50  0001 C CNN
-F 3 "~" H 5900 950 50  0001 C CNN
-	1    5900 950
-	1    0    0    -1
-$EndComp
-Wire Wire Line
-	5500 950  5600 950
-Connection ~ 5500 950
-$Comp
-L power:GND #PWR0152
-U 1 1 5EC13E25
-P 6200 950
-F 0 "#PWR0152" H 6200 700 50  0001 C CNN
-F 1 "GND" H 6200 800 50  0000 C CNN
-F 2 "" H 6200 950 50  0001 C CNN
-F 3 "" H 6200 950 50  0001 C CNN
-	1    6200 950
-	-1   0    0    -1
-$EndComp
+P 6350 1750
+F 0 "SW1" H 6350 1900 50  0000 C CNN
+F 1 "ROM Select" H 6350 1600 50  0000 C CNN
+F 2 "Button_Switch_SMD:SW_DIP_SPSTx01_Slide_6.7x4.1mm_W8.61mm_P2.54mm_LowProfile" H 6350 1750 50  0001 C CNN
+F 3 "~" H 6350 1750 50  0001 C CNN
+	1    6350 1750
+	1    0    0    -1
+$EndComp
+Wire Wire Line
+	5950 1750 6050 1750
+Connection ~ 5950 1750
 $Comp
 L power:GND #PWR0153
@@
 Wire Wire Line
 	6100 3350 6300 3350
+Wire Wire Line
+	6650 1750 6750 1750
+Connection ~ 6750 1750
 $EndSCHEMATC
