File: ROMSIMM8MB.4402B/ROMSIMM.sch (KiCad schematic (older format))
At the start: 39 parts, among them J1 ROM, SW1 ROM Select, U1 MX29LV640, U10 74AHC245, U11 LD1117S33, U12 74LVC1G02GW, U2 MX29LV640, U3 74AHC245, U4 74AHC245, U5 74AHC245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

Commit message: Finished rev. B board
Parts:
- removed SW1: ROM Select, Button_Switch_SMD:SW_DIP_SPSTx01_Slide_6.7x4.1mm_W8.61mm_P2.54mm_LowProfile, symbol Switch:SW_DIP_x01
- removed U11: LD1117S33, stdpads:SOT-223, symbol Regulator_Linear:LD1117S33TR_SOT223
- added R2: 3k3, stdpads:R_0603, symbol Device:R_Small
- added SW1: ROM Sel., stdpads:SW_DIP_SPSTx02_Slide_DSHP02TS_P1.27mm, symbol Switch:SW_DIP_x02
- added U11: XC6206P332MR, stdpads:SOT-23, symbol Regulator_Linear:XC6206PxxxMR
- C1, C10, C11, C12, C13, C14, C15, C2, C3, C4, C5, C6, C7, C8, C9: LCSC Part (none) -> C23630
- H1, H2, H3, H4: footprint stdpads:PasteHole_1.1mm_PTH -> stdpads:PasteHole_1.152mm_NPTH
- R1: footprint stdpads:R_0805 -> stdpads:R_0603; LCSC Part (none) -> C22978
- R3: renamed from R2; footprint stdpads:R_0805 -> stdpads:R_0603; LCSC Part (none) -> C22775
- U1, U2: LCSC Part (none) -> C117907
- U10, U3, U4, U5, U6, U7, U8, U9: LCSC Part (none) -> C132987
- U12: LCSC Part (none) -> C353856
Connections:
- net labels added: RA22sw
- wire segments 82 -> 86
